File: toniebox.kicad_pcb (KiCad board)
At the start: 2 copper layers, 11 parts, among them T11 FDV301N, T4 FDV301N, T5 FDV301N, T6 FDV301N, T7 FDV301N, U1 TLV320DAC3100, U2 CC3200R1M2RGCR, U3 IS25LQ032B-JNLE, U4 MMA8451QT, U8 AP2112K-3.3, U9 AP2120N-1.8

Commit message: readme
Parts:
- moved T7 100.6 mm to (172.0, 131.0), turned to 90 degrees
- moved U3 98.0 mm to (146.0, 127.0), turned to 180 degrees
- moved T6 77.5 mm to (131.0, 66.0)
- moved T5 73.6 mm to (131.0, 72.0)
- moved T4 71.1 mm to (130.9, 60.0)
- moved U1 70.4 mm to (108.0, 61.0)
- moved U2 57.5 mm to (156.0, 103.0), turned to 90 degrees
- moved U9 56.2 mm to (110.0, 72.0), turned to 270 degrees
- moved T11 54.6 mm to (126.0, 73.0), turned to 180 degrees
- moved U8 43.5 mm to (116.9, 72.0), turned to 180 degrees
- moved U4 33.0 mm to (140.0, 68.0)
Other:
- board outline added: 88 x 102 mm
