File: v1-v2/hardware/toniebox-v1v2.kicad_sch (KiCad schematic)
At the start: 133 parts, among them K2 Micro_SD_Card_Det_Hirose_DM3CS, K4 B3B-ZR-SM4-TF, K7 Barrel_Jack_MountingPin, K8 B3B-PH-SM4-TB, K9 B3B-PH-SM4-TB, T11 FDV301N, T360 FDV301N, T4 FDV301N, T5 FDV301N, T6 FDV301N, T7 FDV301N, U1 TLV320DAC3100, U2 CC3200R1M2RGCR, U3 IS25LQ032B-JNLE, U4 MMA8451QT, U7 BQ24400, U8 AP2112K-3.3, U9 AP2120N-1.8

Commit message: wip: schematic
Parts:
- added C58: C, symbol Device:C
- added D301: SS14L, symbol Device:D_Schottky
- added D6: SS14, symbol Device:D_Schottky
- added R305: 0R, symbol Device:R
- added R391: 100k, symbol Device:R
- added R45: 121R, symbol Device:R
- added R48: 221R, symbol Device:R
- added R49: 220k, symbol Device:R
- added R53: 110k, symbol Device:R
- added T2, T3: MMBT3904, Package_TO_SOT_SMD:SOT-23, symbol Transistor_BJT:MMBT3904
- added U300: LM3485MM, Package_SO:VSSOP-8_3.0x3.0mm_P0.65mm, symbol Regulator_Controller:LM3478MM
- added U6: AP2114H-3.3TRG1, Package_TO_SOT_SMD:SOT-223-3_TabPin2, symbol Regulator_Linear:AP1117-33
Connections:
- net GND: now also R55.1, TP6.1, U7.2 (VSS), C58.2, R48.2, R53.1
- net at TP75.1: now also R305.2, U300.8 (V_{IN})
- net at TP300.1: now also D301.2 (A), U300.1 (ISENSE)
- net at TP42.1: now also U7.4 (BAT), C58.1, R391.2
- net BAT+: now reaches K8.3, TP38.1
- net BAT+: now also R49.1
- net at TP301.1: now also D6.1 (K), R305.1
- net +3V3: now reaches U2.10 (VIN_IO1)
- net +3V3: now also U6.2 (VO)
- net at U7.8 (MOD): now also T3.1 (B)
- new net: R45.1, T2.2 (E)
- new net: R391.1, R49.2, R53.2
- new net: D301.1 (K), U6.3 (VI)
- new net: R45.2, T3.3 (C)
- new net: R48.1, T3.2 (E)
Other:
- note added: "9V, 1.5A"
- moved on the sheet: K7, K9, R55, TP11, TP17, TP18, TP300, TP301, TP38, TP42, TP55, TP6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
